File: hw/picocart64_v1_lite/picocart64_v1_lite.kicad_sch (KiCad schematic)
At the start: 10 parts, among them J1 Conn_01x04, J2 Conn_01x07, J3 Conn_01x02, J4 Conn_01x01, J5 Conn_01x01, Q1 BSS84, U1 Pico, U4 N64-Cartridge

Commit message: bom prep
Parts:
- J1: LCSC (none) -> C390680
- J2: LCSC (none) -> C225482
- J3, J4, J5, JP1, U1, U4: now left out of the parts list
- Q1: LCSC (none) -> C114481
- R1: LCSC (none) -> C22936
Changed lines of the file:
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@@
   )
   (symbol (lib_id "Jumper:SolderJumper_2_Open") (at 72.39 55.88 0) (unit 1)
-    (in_bom yes) (on_board yes)
+    (in_bom no) (on_board yes)
     (property "Reference" "JP1" (id 0) (at 77.47 54.61 0))
     (property "Value" "SolderJumper_2_Open" (id 1) (at 103.505 55.245 0)
@@
       (effects (font (size 1.27 1.27)) (justify left) hide)
     )
+    (property "LCSC" "C114481" (id 4) (at 85.09 26.67 90)
+      (effects (font (size 1.27 1.27)) hide)
+    )
     (pin "1")
     (pin "2")
@@
   )
   (symbol (lib_id "Connector_Generic:Conn_01x02") (at 124.46 151.13 0) (unit 1)
-    (in_bom yes) (on_board yes) (fields_autoplaced)
+    (in_bom no) (on_board yes) (fields_autoplaced)
     (property "Reference" "J3" (id 0) (at 127 151.1299 0)
       (effects (font (size 1.27 1.27)) (justify left))
@@
   )
   (symbol (lib_id "raspberrypi_pico:Pico") (at 48.26 72.39 0) (unit 1)
-    (in_bom yes) (on_board yes) (fields_autoplaced)
+    (in_bom no) (on_board yes) (fields_autoplaced)
     (property "Reference" "U1" (id 0) (at 48.26 41.91 0))
     (property "Value" "Pico" (id 1) (at 48.26 44.45 0))
@@
   )
   (symbol (lib_id "n64-cartridge:N64-Cartridge") (at 237.49 55.88 0) (unit 1)
-    (in_bom yes) (on_board yes) (fields_autoplaced)
+    (in_bom no) (on_board yes) (fields_autoplaced)
     (property "Reference" "U4" (id 0) (at 236.855 17.78 0)
       (effects (font (size 1.524 1.524)))
@@
   )
   (symbol (lib_id "Connector_Generic:Conn_01x01") (at 35.56 148.59 180) (unit 1)
-    (in_bom yes) (on_board yes)
+    (in_bom no) (on_board yes)
     (property "Reference" "J5" (id 0) (at 31.75 148.59 0))
     (property "Value" "Conn_01x01" (id 1) (at 22.86 148.59 0))
@@
     )
     (property "Datasheet" "~" (id 3) (at 76.2 151.13 0)
+      (effects (font (size 1.27 1.27)) hide)
+    )
+    (property "LCSC" "C225482" (id 4) (at 76.2 151.13 0)
       (effects (font (size 1.27 1.27)) hide)
     )
@@
   )
   (symbol (lib_id "Connector_Generic:Conn_01x01") (at 35.56 143.51 180) (unit 1)
-    (in_bom yes) (on_board yes)
+    (in_bom no) (on_board yes)
     (property "Reference" "J4" (id 0) (at 31.75 143.51 0))
     (property "Value" "Conn_01x01" (id 1) (at 22.86 143.51 0))
@@
     )
     (property "Datasheet" "~" (id 3) (at 91.44 34.29 0)
+      (effects (font (size 1.27 1.27)) hide)
+    )
+    (property "LCSC" "C22936" (id 4) (at 91.44 34.29 90)
       (effects (font (size 1.27 1.27)) hide)
     )
@@
       (effects (font (size 1.27 1.27)) hide)
     )
+    (property "LCSC" "C390680" (id 4) (at 69.85 146.05 0)
+      (effects (font (size 1.27 1.27)) hide)
+    )
